File: VoyaLite.kicad_sch (KiCad schematic)
At the start: 125 parts

Commit message: change things
Parts:
- added C32, C34: 10u, Capacitor_SMD:C_0805_2012Metric_Pad1.18x1.45mm_HandSolder, symbol Device:C_Small
- added C33, C40: 100n, Capacitor_SMD:C_0805_2012Metric_Pad1.18x1.45mm_HandSolder, symbol Device:C_Small
- added C35: 22uF, Capacitor_SMD:C_0805_2012Metric_Pad1.18x1.45mm_HandSolder, symbol Device:C_Small
- added C36: 1u, symbol Device:C_Small
- added C37, C38, C39: 4u7, symbol Device:C_Small
- added D32, D33, D34, D35, D36, D37, D38, D39, D40, D41, D42, D43, D44, D45, D46, D47, D48, D49, D50, D51, D52, D53, D54, D55, D56, D57, D58, D59, D60, D61, D62: D, Diode_SMD:D_MiniMELF, symbol Diode:LL4148
- added J1: Conn_01x02_Socket, Connector_JST:JST_ZH_B2B-ZR_1x02_P1.50mm_Vertical, symbol Connector:Conn_01x02_Socket
- added J2: Screw_Terminal_01x02, symbol Connector:Screw_Terminal_01x02
- added J3: USB_C_Receptacle_USB2.0_16P, symbol Connector:USB_C_Receptacle_USB2.0_16P
- added JP1: SolderJumper_2_Open, Jumper:SolderJumper-2_P1.3mm_Open_RoundedPad1.0x1.5mm, symbol Jumper:SolderJumper_2_Open
- added L2: 2u2H, Inductor_SMD:L_Vishay_IFSC-1515AH_4x4x1.8mm, symbol Device:L_Small
- added NT1: NetTie_2, NetTie:NetTie-2_THT_Pad0.3mm, symbol Device:NetTie_2
- added R1: 1.18k, symbol Device:R_Small
- added R2: 1.13k, symbol Device:R_Small
- added R3, R4: 51K, symbol Device:R_Small
- added SW1: SW_SPDT_312, Button_Switch_SMD:SW_SPDT_PCM12, symbol Switch:SW_SPDT_312
- added U1: RP604K501A-TR, Library_Pia:DFN(PL)2730-12, symbol RT-Library-Kicad:RP6040-12
- added U2: E73-2G4M08S1C, E73-2G4M08S1C:E73-2G4M08S1C, symbol RT-Library-Kicad:E73-2G4M08S1C
- added U3: BQ24075RGT, Package_DFN_QFN:VQFN-16-1EP_3x3mm_P0.5mm_EP1.6x1.6mm, symbol Battery_Management:BQ24075RGT
- LED1, LED10, LED11, LED12, LED13, LED14, LED15, LED16, LED17, LED18, LED19, LED2, LED20, LED21, LED22, LED23, LED24, LED25, LED26, LED27, LED28, LED29, LED3, LED30, LED31, LED4, LED5, LED6, LED7, LED8, LED9: footprint (none) -> MX_Alps_Hybrid:SK6803-MINI-E_pia
- S1, S10, S11, S12, S13, S14, S15, S16, S17, S18, S19, S2, S20, S21, S22, S23, S24, S25, S26, S27, S28, S29, S3, S30, S31, S4, S5, S6, S7, S8, S9: footprint (none) -> KeySwitches_DalePrice:Kailh_socket_PG1350_reversible
- SuperMiniNRF53840: renamed from MCU1; footprint (none) -> Library_Pia:supermini NRF52840 superflat
Connections:
- net GND: now also C32.2, C33.2, C34.2, C35.2, C36.2, C37.2, C38.2, C39.2, C40.2, J2.2 (Pin_2), NT1.1, R1.2, R2.2, R3.2, R4.2, U1.3,4,9,10,13 (PGND), U2.21 (GND@2), U2.24 (GND@3), U2.5 (GND@1), U3.14 (TMR), U3.4 (~{CE}), U3.6 (EN1)
- net LED: now also SuperMiniNRF53840.22 (VCC), C34.1, JP1.1 (A), U1.1 (AVIN), U1.12 (PVIN); no longer LED1.3 (DIN), SuperMiniNRF53840.14 (600)
- net r1: now also D32.1 (K), D36.1 (K), D41.1 (K), D46.1 (K), D51.1 (K), D56.1 (K), D61.1 (K)
- net r2: now also D33.1 (K), D37.1 (K), D42.1 (K), D47.1 (K), D52.1 (K), D57.1 (K), D62.1 (K)
- net r3: now also D34.1 (K), D38.1 (K), D43.1 (K), D48.1 (K), D53.1 (K), D58.1 (K)
- net r4: now also D35.1 (K), D39.1 (K), D44.1 (K), D49.1 (K), D54.1 (K), D59.1 (K)
- net r5: now also D40.1 (K), D45.1 (K), D50.1 (K), D55.1 (K), D60.1 (K)
- net at D10.2 (A), S10.2: now also D45.2 (A)
- net at D18.2 (A), S18.2: now also D47.2 (A)
- net at D3.2 (A), S3.2: now also D34.2 (A)
- net at D21.2 (A), S21.2: now also D54.2 (A)
- net at D29.2 (A), S29.2: now also D56.2 (A)
- net at D14.2 (A), S14.2: now also D41.2 (A)
- net at D17.2 (A), S17.2: now also D48.2 (A)
- net at D8.2 (A), S8.2: now also D39.2 (A)
- net at D23.2 (A), S23.2: now also D52.2 (A)
- net at D28.2 (A), S28.2: now also D57.2 (A)
- net at D11.2 (A), S11.2: now also D44.2 (A)
- net at D4.2 (A), S4.2: now also D35.2 (A)
- net at D20.2 (A), S20.2: now also D55.2 (A)
- net at D1.2 (A), S1.2: now also D32.2 (A)
- net at D15.2 (A), S15.2: now also D50.2 (A)
- net at D27.2 (A), S27.2: now also D58.2 (A)
- net at D24.2 (A), S24.2: now also D51.2 (A)
- net at D6.2 (A), S6.2: now also D37.2 (A)
- net -BATT: now reaches SuperMiniNRF53840.1 (B-)
- net -BATT: now also J1.2 (Pin_2)
- net +3V8: now reaches SuperMiniNRF53840.25 (RAW)
- net +3V8: now also SuperMiniNRF53840.26 (B+), C32.1, C33.1, C37.1, SW1.1 (B), U3.10 (OUT), U3.11 (OUT)
- net at D13.2 (A), S13.2: now also D42.2 (A)
- net at D5.2 (A), S5.2: now also D36.2 (A)
- net at D25.2 (A), S25.2: now also D60.2 (A)
- net at D9.2 (A), S9.2: now also D40.2 (A)
- net at D2.2 (A), S2.2: now also D33.2 (A)
- net at D31.2 (A), S31.2: now also D62.2 (A)
- net at D19.2 (A), S19.2: now also D46.2 (A)
- net at D30.2 (A), S30.2: now also D61.2 (A)
- net at D7.2 (A), S7.2: now also D38.2 (A)
- net at D26.2 (A), S26.2: now also D59.2 (A)
- net at D22.2 (A), S22.2: now also D53.2 (A)
- net at D12.2 (A), S12.2: now also D43.2 (A)
- net at D16.2 (A), S16.2: now also D49.2 (A)
- new net: C39.1, C40.1, U2.19 (VDD)
- new net: J3.A7 (D-), J3.B7 (D-), U2.29 (DM)
- new net: J3.A6 (D+), J3.B6 (D+), U2.31 (DP)
- new net: NT1.2, U1.5 (AGND)
- new net: J3.B5 (CC2), R4.1
- new net: R1.1, U3.12 (ILIM)
- new net: R2.1, U3.16 (ISET)
- new net: U3.17 (VSS), U3.8 (VSS)
- new net: J3.A5 (CC1), R3.1
- new net: L2.1, U1.11 (BULX)
- new net: L2.2, U1.8 (BOLX)
- new net: J3.A1 (GND), J3.A12 (GND), J3.B1 (GND), J3.B12 (GND)
- new net +BATT: J1.1 (Pin_1), SW1.3 (A)
- new net Bat+: C38.1, J2.1 (Pin_1), U3.2 (BAT), U3.3 (BAT), U3.5 (EN2)
- new net Boost_EN: SuperMiniNRF53840.14 (600), U1.2 (CE)
- new net LED_IN: C35.1, JP1.2 (B), LED1.3 (DIN), U1.6 (VFB), U1.7 (VOUT)
- new net VBUS: C36.1, J3.A4 (VBUS), J3.A9 (VBUS), J3.B4 (VBUS), J3.B9 (VBUS), U2.27 (VBUS), U3.13 (IN)
Other:
- note added: "Batterien: https://www.amazon.de/Batterien-Wiederaufladbare-Fernbedienung-Controller-Blitzlichter/dp/B074V2QVC3/ref=sr_1_3?__mk_de_DE"
- moved on the sheet: S1, S10, S11, S12, S13, S14, S15, S16, S17, S18, S19, S2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
