File: VoyaLite.kicad_sch (KiCad schematic)
At the start: 45 parts, among them J1 Conn_01x01_Pin, J2 Conn_01x01_Pin, Q1 NTJD1155LT1G, Q2 NTJD1155LT1G, U6 XIAO-NRF82840-Plus

Commit message: add final changes
Parts:
- added C2: 1u, Capacitor_SMD:C_0402_1005Metric_Pad0.74x0.62mm_HandSolder, symbol Device:C_Small
- added C3: 100n, Capacitor_SMD:C_0402_1005Metric_Pad0.74x0.62mm_HandSolder, symbol Device:C_Small
Connections:
- net +BATT: now also C2.1, C3.1; no longer U6.12 (P0.31/BAT/D16)
- net GND: now also U6.22 (GND), C2.2, C3.2
Other:
- moved on the sheet: BT1, J1, J2
