File: VoyaLite_Right.kicad_pcb (KiCad board)
At the start: 2 copper layers, 153 x 143 mm, 50 parts, among them J1 Conn_01x01_Pin, J2 Conn_01x01_Pin, Q1 NTJD1155LT1G, Q2 NTJD1155LT1G, U6 XIAO-NRF82840-Plus

Commit message: add new production files
Parts:
- removed G***: LOGO, Pia_Lib:Logo-kuh
- removed kibuzzard-691072A3: G***, kibuzzard-691072A3
- removed kibuzzard-691072AF: G***, kibuzzard-691072AF
